File: v1/ahokore.kicad_pcb (KiCad board)
At the start: 2 copper layers, 248.2 x 100 mm, 87 parts, among them SW1 SW_SPDT, SW10 SW_Push, SW11 SW_Push, SW12 SW_Push, SW13 SW_Push, SW14 SW_Push, SW15 SW_Push, SW16 SW_Push, SW17 SW_Push, SW18 SW_Push, SW19 SW_Push, SW2 SW_Push, SW20 SW_Push, SW21 SW_Push, SW22 SW_Push, SW23 SW_Push, SW24 SW_Push, SW25 SW_Push, SW26 SW_Push, SW27 SW_Push, SW28 SW_Push, SW29 SW_Push, SW3 SW_Push, SW30 SW_Push, SW31 SW_Push, SW32 SW_Push, SW33 SW_Push, SW34 SW_Push, SW35 SW_Push, SW36 SW_Push, SW37 SW_Push, SW38 SW_Push, SW4 SW_Push, SW5 SW_Push, SW6 SW_Push, SW7 SW_Push, SW8 SW_Push, SW9 SW_Push, U1 ProMicro

Commit message: update pcb kikads
Parts:
- removed G***: LOGO, custom-parts:astro
- removed G***: LOGO, custom-parts:logo6
- removed G***: LOGO, custom-parts:logocopper
- removed the REF** at (90.3, -20.6)
- removed the REF** at (-89.7, -20.6)
- removed the REF** at (-109.7, -85.5)
- removed the REF** at (110.3, -85.5)
- moved BT1 15.0 mm to (-1.98, -38.0)
- moved SW1 15.0 mm to (13.6, -77.5)
- moved SW2 15.0 mm to (-13.5, -70.0)
- moved U1 15.0 mm to (0.33, -60.5)
- moved REF** 10.0 mm to (20.3, -60.5)
- moved REF** 10.0 mm to (-19.7, -60.5)
Routing:
- net COL9: track 207.2 -> 175.4 mm
- net COL8: track 180.6 -> 153.0 mm
- net COL7: track 181.1 -> 161.6 mm
- net ROW2: track 253.4 -> 234.6 mm
- net COL2: track 148.3 -> 136.2 mm
- net ROW0: track 287.5 -> 276.7 mm
- net ROW3: track 188.3 -> 177.5 mm
- net COL4: track 112.3 -> 103.7 mm
- net ROW1: track 253.5 -> 245.1 mm
- net COL6: track 153.5 -> 145.6 mm
- net COL3: track 122.4 -> 114.9 mm
- net COL5: track 129.8 -> 125.6 mm
- net COL1: track 139.9 -> 137.8 mm
- net COL0: track 159.1 -> 157.5 mm
Other:
- board outline removed
- net class Default removed
- net class Power removed
- board text removed: "Ahokore V1"
- board text removed: "Licensed under CERN-OHL-P v2."
- board text removed: "designed alongside Bonsa"
- board text removed: "powered by ZMK"
- board text removed: "thank you everyone for the help"
